File: kicad/diy_led_spot/diy_led_spot.kicad_pcb (KiCad board)
At the start: 2 copper layers, 50.5 x 47.5 mm, 33 parts, among them Q1 AO3400A_C347475, U1 DCDCStepDown, U2 PT4115, U3 ESP32-C3_SUPERMINI_SMD, U4 MT3608, U5 110kΩ

Commit message: kicad: save current PCB/schematic state
Parts:
- D4: value 1N4148W-7-F -> SS36; footprint easyeda2kicad:SOD-123_L2.7-W1.6-LS3.7-RD-1 -> easyeda2kicad:SMA_L4.3-W2.6-LS5.2-RD
- TEMP1: value MX1.25-2P -> BX-XH2.54-2PZZ; footprint easyeda2kicad:CONN-SMD_2P-P1.25_XUNPU_WAFER-MX1.25-2PWB -> easyeda2kicad:CONN-TH_2P-P2.50_BX-XH2.54-2PZZ
- moved R1 3.82 mm to (123.5, 105.2)
- moved D4 2.35 mm to (126.8, 96.2)
- moved C3 2.24 mm to (123.5, 103.0)
- moved TEMP1 1.23 mm to (114.5, 102.5)
- moved IN+1 0.50 mm to (115.5, 71.0)
