File: kicad/diy_led_spot/diy_led_spot_step3.kicad_pcb (KiCad board)
At the start: 2 copper layers, 50.5 x 47.5 mm, 37 parts, among them Q1 AO3400A_C347475, U1 DCDCStepDown, U2 PT4115, U3 ESP32-C3_SUPERMINI_SMD, U4 MT3608, U5 110kΩ

Commit message: feat: enhance documentation and improve spots discoverability
Parts:
- renumbered -LED+1 to +LED-, U3 to ESP32
Changed lines of the file:
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@@
 		(layer "F.Cu")
 		(at 150.5 96 180)
-		(property "Reference" "U3"
-			(at -5.715 -13.6525 0)
+		(property "Reference" "ESP32"
+			(at 0 0 0)
 			(layer "F.SilkS")
 			(effects
@@
 		(layer "F.Cu")
 		(at 114.5 85 -90)
-		(property "Reference" "-LED+1"
+		(property "Reference" "+LED-"
 			(at 0 -4.5 90)
 			(layer "F.SilkS")
@@
 	)
 	(segment
-		(start 146.2 73.8)
-		(end 147 73.8)
+		(start 142.8 81.2)
+		(end 151.3 81.2)
 		(width 0.3)
 		(layer "F.Cu")
@@
 	)
 	(segment
-		(start 144 75.3)
-		(end 140.9 78.4)
+		(start 146.2 73.8)
+		(end 147 73.8)
 		(width 0.3)
 		(layer "F.Cu")
@@
 	)
 	(segment
-		(start 151.3 81.2)
-		(end 155.5 77)
+		(start 141 79.3)
+		(end 141 79.4)
 		(width 0.3)
 		(layer "F.Cu")
@@
 	)
 	(segment
-		(start 141 80.2)
-		(end 141 84.1)
-		(width 0.3)
-		(layer "F.Cu")
-		(net 11)
-	)
-	(segment
-		(start 140.9 80.1)
-		(end 141 80.2)
-		(width 0.3)
-		(layer "F.Cu")
-		(net 11)
-	)
-	(segment
-		(start 140.9 78.4)
-		(end 140.9 80.1)
+		(start 151.3 81.2)
+		(end 155.5 77)
 		(width 0.3)
 		(layer "F.Cu")
@@
 	)
 	(segment
-		(start 142.8 81.2)
-		(end 151.3 81.2)
+		(start 144 75.3)
+		(end 141 78.3)
+		(width 0.3)
+		(layer "F.Cu")
+		(net 11)
+	)
+	(segment
+		(start 141 78.3)
+		(end 141 84.1)
 		(width 0.3)
 		(layer "F.Cu")
@@
 	)
 	(segment
-		(start 140.9 79.3)
+		(start 141 79.4)
 		(end 142.8 81.2)
 		(width 0.3)
@@
 	)
 	(segment
-		(start 155.9 76.1)
-		(end 156.1 76.1)
+		(start 154.2 74.4)
+		(end 153.1 75.5)
 		(width 0.3)
 		(layer "F.Cu")
@@
 	)
 	(segment
-		(start 154.2 74.4)
-		(end 153.1 75.5)
+		(start 156.5 87.1)
+		(end 156.5 104.4)
 		(width 0.3)
 		(layer "F.Cu")
@@
 	)
 	(segment
-		(start 158 105.9)
-		(end 158.5 105.9)
+		(start 156.25 75.75)
+		(end 157.5 77)
 		(width 0.3)
 		(layer "F.Cu")
@@
 	)
 	(segment
-		(start 157.5 79.1)
-		(end 157.5 86.1)
+		(start 157.5 86.1)
+		(end 156.5 87.1)
 		(width 0.3)
 		(layer "F.Cu")
@@
 	)
 	(segment
-		(start 157.5 86.1)
-		(end 156.5 87.1)
+		(start 157.5 77)
+		(end 157.5 86.1)
 		(width 0.3)
 		(layer "F.Cu")
@@
 	)
 	(segment
-		(start 157.4 79)
-		(end 157.5 79.1)
+		(start 155.55 75.75)
+		(end 156.25 75.75)
 		(width 0.3)
 		(layer "F.Cu")
@@
 	)
 	(segment
-		(start 156.5 104.4)
-		(end 158 105.9)
+		(start 154.2 74.4)
+		(end 155.55 75.75)
 		(width 0.3)
 		(layer "F.Cu")
@@
 	)
 	(segment
-		(start 153.1 75.5)
-		(end 152.9 75.5)
+		(start 156.5 104.4)
+		(end 158 105.9)
 		(width 0.3)
 		(layer "F.Cu")
@@
 	)
 	(segment
-		(start 151.3 75.5)
-		(end 151 75.2)
+		(start 153.1 75.5)
+		(end 152.9 75.5)
 		(width 0.3)
 		(layer "F.Cu")
@@
 	)
 	(segment
-		(start 156.1 76.1)
-		(end 158.2 78.2)
+		(start 151.3 75.5)
+		(end 151 75.2)
 		(width 0.3)
 		(layer "F.Cu")
@@
 	)
 	(segment
-		(start 158.2 78.2)
-		(end 157.4 79)
+		(start 158 105.9)
+		(end 158.5 105.9)
 		(width 0.3)
 		(layer "F.Cu")
@@
 	)
 	(segment
-		(start 156.5 87.1)
-		(end 156.5 104.4)
-		(width 0.3)
-		(layer "F.Cu")
-		(net 17)
-	)
-	(segment
 		(start 148.5 75.2)
 		(end 148.5 75.25)
 		(width 0.3)
 		(layer "F.Cu")
-		(net 17)
-	)
-	(segment
-		(start 154.2 74.4)
-		(end 155.9 76.1)
-		(width 0.3)
-		(layer "F.Cu")
